File: lineScope.kicad_pcb (KiCad board)
At the start: 2 copper layers, 0 parts

Commit message: Route pcb
Parts:
- added C1: 100n, Capacitor_SMD:C_0603_1608Metric, F.Cu at (119.2, 88.0)
- added C10: 1u, Capacitor_SMD:C_0603_1608Metric, F.Cu at (144.3, 77.0)
- added C11: 470u, Capacitor_SMD:CP_Elec_10x10.5, F.Cu at (193.8, 75.9)
- added C12: 100n, Capacitor_SMD:C_0603_1608Metric, F.Cu at (186.1, 67.2)
- added C13: 100n, Capacitor_SMD:C_0603_1608Metric, F.Cu at (186.3, 73.9)
- added C15: 100n, Capacitor_SMD:C_0603_1608Metric, F.Cu at (186.3, 77.1)
- added C18: 470u, Capacitor_SMD:CP_Elec_10x10.5, F.Cu at (107.6, 73.6)
- added C19: 100n, Capacitor_SMD:C_0603_1608Metric, F.Cu at (117.3, 72.6)
- added C2: 1u, Capacitor_SMD:C_0603_1608Metric, F.Cu at (125.6, 88.0)
- added C20: 100n, Capacitor_SMD:C_0603_1608Metric, F.Cu at (117.3, 69.6)
- added C21: 1u, Capacitor_SMD:C_0603_1608Metric, F.Cu at (133.0, 68.5)
- added C22: 1u, Capacitor_SMD:C_0603_1608Metric, F.Cu at (144.0, 70.1)
- added C23: 100n, Capacitor_SMD:C_0603_1608Metric, F.Cu at (144.0, 68.5)
- added C3: 1u, Capacitor_SMD:C_0603_1608Metric, F.Cu at (124.0, 88.0)
- added C4: 1u, Capacitor_SMD:C_0603_1608Metric, F.Cu at (123.8, 76.8)
- added C5: 1u, Capacitor_SMD:C_0603_1608Metric, F.Cu at (125.7, 76.8)
- added C6: 100n, Capacitor_SMD:C_0603_1608Metric, F.Cu at (137.9, 88.0)
- added C7: 1u, Capacitor_SMD:C_0603_1608Metric, F.Cu at (144.3, 88.0)
- added C8: 1u, Capacitor_SMD:C_0603_1608Metric, F.Cu at (142.7, 88.0)
- added C9: 1u, Capacitor_SMD:C_0603_1608Metric, F.Cu at (142.6, 77.0)
- added D10: ESD3B15WS, Diode_SMD:D_SOD-323_HandSoldering, F.Cu at (186.3, 94.1)
- added D11: ESD3B15WS, Diode_SMD:D_SOD-323_HandSoldering, F.Cu at (121.6, 66.8)
- added D12: ESD3B15WS, Diode_SMD:D_SOD-323_HandSoldering, F.Cu at (140.6, 66.8)
- added D2: MB2S, Package_TO_SOT_SMD:TO-269AA, F.Cu at (188.7, 61.4)
- added D5: MB2S, Package_TO_SOT_SMD:TO-269AA, F.Cu at (110.8, 63.8)
- added D6: ESD3B15WS, Diode_SMD:D_SOD-323_HandSoldering, F.Cu at (116.3, 94.1)
- added D7: LL103A, Diode_SMD:D_MiniMELF, B.Cu at (165.5, 85.3)
- added D8: ESD3B15WS, Diode_SMD:D_SOD-323_HandSoldering, F.Cu at (151.3, 94.1)
- added D9: LL103A, Diode_SMD:D_MiniMELF, B.Cu at (165.3, 75.2)
- added H1: M3, MountingHole:MountingHole_3.2mm_M3_Pad, F.Cu at (105.0, 55.0)
- added H2: M3, MountingHole:MountingHole_3.2mm_M3_Pad, F.Cu at (195.0, 55.0)
- added H3: M3, MountingHole:MountingHole_3.2mm_M3_Pad, F.Cu at (195.0, 95.0)
- added H4: M3, MountingHole:MountingHole_3.2mm_M3_Pad, F.Cu at (105.0, 95.0)
- added J1: Conn_01x02, Connector_JST:JST_XH_B2B-XH-A_1x02_P2.50mm_Vertical, F.Cu at (197.0, 61.6)
- added J2: Conn_01x02, Connector_JST:JST_XH_B2B-XH-A_1x02_P2.50mm_Vertical, F.Cu at (103.0, 65.0)
- added J3: Conn_01x03, Connector_PinSocket_2.54mm:PinSocket_1x03_P2.54mm_Horizontal, F.Cu at (112.5, 98.6)
- added J4: Conn_01x03, Connector_PinSocket_2.54mm:PinSocket_1x03_P2.54mm_Horizontal, F.Cu at (147.5, 98.6)
- added J5: Conn_01x03, Connector_PinSocket_2.54mm:PinSocket_1x03_P2.54mm_Horizontal, F.Cu at (182.5, 98.6)
- added J7: Conn_Coaxial, Connector_Coaxial:BNC_Amphenol_B6252HB-NPP3G-50_Horizontal, F.Cu at (124.3, 63.0)
- added J8: Conn_Coaxial, Connector_Coaxial:BNC_Amphenol_B6252HB-NPP3G-50_Horizontal, F.Cu at (143.3, 63.0)
- added J9: Conn_01x04, Connector_JST:JST_XH_B4B-XH-A_1x04_P2.50mm_Vertical, F.Cu at (166.7, 53.5)
- added K1: HE721A0500, Koszalix_Relays:HE721A050, F.Cu at (165.3, 81.5)
- added K2: HE721A0500, Koszalix_Relays:HE721A050, F.Cu at (165.3, 71.4)
- added Q1: BC847, Package_TO_SOT_SMD:SOT-23, F.Cu at (164.3, 64.2)
- added Q2: BC847, Package_TO_SOT_SMD:SOT-23, F.Cu at (171.8, 64.3)
- added R1: 10k, Resistor_SMD:R_0603_1608Metric, F.Cu at (120.8, 88.0)
- added R10: 0R, Resistor_SMD:R_0603_1608Metric, F.Cu at (195.8, 90.6)
- added R11: 0R, Resistor_SMD:R_0603_1608Metric, F.Cu at (116.8, 92.3)
- added R12: 10k, Resistor_SMD:R_0603_1608Metric, F.Cu at (113.7, 92.3)
- added R13: 0R, Resistor_SMD:R_0603_1608Metric, F.Cu at (151.8, 92.3)
- added R14: 10k, Resistor_SMD:R_0603_1608Metric, F.Cu at (148.7, 92.3)
- added R15: 0R, Resistor_SMD:R_0603_1608Metric, F.Cu at (186.8, 92.3)
- added R16: 10k, Resistor_SMD:R_0603_1608Metric, F.Cu at (183.7, 92.3)
- added R17: 470R, Resistor_SMD:R_0603_1608Metric, F.Cu at (169.2, 64.7)
- added R18: 51R, Resistor_SMD:R_0603_1608Metric, F.Cu at (125.3, 66.8)
- added R19: 1k, Resistor_SMD:R_0603_1608Metric, F.Cu at (133.0, 70.1)
- added R2: 10k, Resistor_SMD:R_0603_1608Metric, F.Cu at (122.4, 88.0)
- added R20: 1k, Resistor_SMD:R_0603_1608Metric, F.Cu at (133.0, 71.7)
- added R21: 51R, Resistor_SMD:R_0603_1608Metric, F.Cu at (144.3, 66.8)
- added R22: 1k, Resistor_SMD:R_0603_1608Metric, F.Cu at (144.0, 71.7)
- added R23: 1k, Resistor_SMD:R_0603_1608Metric, F.Cu at (144.0, 73.2)
- added R24: 0R, Resistor_SMD:R_0603_1608Metric, F.Cu at (105.9, 90.5)
- added R25: 10k, Resistor_SMD:R_0603_1608Metric, F.Cu at (174.4, 64.7)
- added R3: 10k, Resistor_SMD:R_0603_1608Metric, F.Cu at (139.5, 88.0)
- added R4: 10k, Resistor_SMD:R_0603_1608Metric, F.Cu at (141.1, 88.0)
- added R5: 10k, Resistor_SMD:R_0603_1608Metric, F.Cu at (166.9, 64.7)
- added R6: 470R, Resistor_SMD:R_0603_1608Metric, F.Cu at (161.7, 64.6)
- added R7: 0R, Resistor_SMD:R_0603_1608Metric, F.Cu at (109.3, 55.8)
- added R8: 4k7, Resistor_SMD:R_0603_1608Metric, F.Cu at (186.3, 75.5)
- added R9: 0R, Resistor_SMD:R_0603_1608Metric, F.Cu at (190.5, 55.8)
- added REF**: OSHW-Logo2_7.3x6mm_SilkScreen, Symbol:OSHW-Logo2_7.3x6mm_SilkScreen, F.Cu at (142.0, 96.0)
- added REF**: WEEE-Logo_4.2x6mm_SilkScreen, Symbol:WEEE-Logo_4.2x6mm_SilkScreen, F.Cu at (158.4, 61.0)
- added REF**: ESD-Logo_6.6x6mm_SilkScreen, Symbol:ESD-Logo_6.6x6mm_SilkScreen, F.Cu at (158.6, 53.8)
- added RV1: MCVZ0603M180AGT, Resistor_SMD:R_0603_1608Metric_Pad0.98x0.95mm_HandSolder, F.Cu at (186.8, 65.0)
- added RV3: MCVZ0603M180AGT, Resistor_SMD:R_0603_1608Metric_Pad0.98x0.95mm_HandSolder, F.Cu at (115.6, 64.0)
- added RV4: MCVZ0603M180AGT, Resistor_SMD:R_0603_1608Metric_Pad0.98x0.95mm_HandSolder, F.Cu at (116.7, 95.9)
- added RV5: MCVZ0603M180AGT, Resistor_SMD:R_0603_1608Metric_Pad0.98x0.95mm_HandSolder, F.Cu at (151.7, 95.9)
- added RV6: MCVZ0603M180AGT, Resistor_SMD:R_0603_1608Metric_Pad0.98x0.95mm_HandSolder, F.Cu at (186.7, 95.9)
- added TP1: TestPoint, TestPoint:TestPoint_Pad_D1.0mm, F.Cu at (181.0, 79.0)
- added TP2: TestPoint, TestPoint:TestPoint_Pad_D1.0mm, F.Cu at (181.0, 72.0)
- added TP3: TestPoint, TestPoint:TestPoint_Pad_D1.0mm, F.Cu at (181.0, 75.5)
- added TP4: TestPoint, TestPoint:TestPoint_Pad_D1.0mm, F.Cu at (125.4, 69.6)
- added TP5: TestPoint, TestPoint:TestPoint_Pad_D1.0mm, F.Cu at (127.6, 69.6)
- added U1: ADuM3190, Package_SO:QSOP-16_3.9x4.9mm_P0.635mm, F.Cu at (123.4, 82.6)
- added U2: ADuM3190, Package_SO:QSOP-16_3.9x4.9mm_P0.635mm, F.Cu at (142.2, 82.5)
- added U3: L78L09_SOT89, Package_TO_SOT_SMD:SOT-89-3, F.Cu at (184.9, 70.5)
- added U4: LM4040DBZ-2.0, Package_TO_SOT_SMD:SOT-23, F.Cu at (185.8, 79.7)
- added U5: L78L09_SOT89, Package_TO_SOT_SMD:SOT-89-3, F.Cu at (121.8, 71.1)
- added U6: LM358, Package_SO:SO-8_3.9x4.9mm_P1.27mm, F.Cu at (138.5, 71.0)
Routing:
- net VCC2: track 0.00 -> 192.3 mm, vias 0 -> 3
- net VREF2: track 0.00 -> 108.9 mm, vias 0 -> 4
- net VCC1: track 0.00 -> 76.3 mm, vias 0 -> 4
- net /Isolators/IN.I: track 0.00 -> 38.9 mm
- net Net-(K1-Pad7): track 0.00 -> 37.0 mm
- net Net-(K2-Pad7): track 0.00 -> 36.4 mm
- net GND2: track 0.00 -> 31.1 mm, vias 0 -> 221
- net Net-(D7-A): track 0.00 -> 28.2 mm, vias 0 -> 1
- net Net-(D2-+): track 0.00 -> 28.1 mm
- net /Isolators/VV: track 0.00 -> 21.2 mm
- net Net-(D5-+): track 0.00 -> 20.9 mm
- net GND1: track 0.00 -> 17.3 mm, vias 0 -> 61
- net Net-(D9-A): track 0.00 -> 16.0 mm, vias 0 -> 1
- net /Isolators/IN.V: track 0.00 -> 11.0 mm
- net Net-(J9-Pin_3): track 0.00 -> 10.8 mm
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- added copper zone on B.Cu, net GND1
- added copper zone on F.Cu, net GND1
- added copper zone on B.Cu, net GND2
- added copper zone on F.Cu, net GND2
Other:
- board outline added: 100 x 50 mm
- board text added: "AC1"
- board text added: "AC2"
- board text added: "CONTROL"
- board text added: "CURRENT PROBE H"
- board text added: "CURRENT PROBE L"
- board text added: "VOLTAGE PROBE"
- board text added: "lineScope Isolators Rev 1.0.0 03/2024"
