File: lineScope.kicad_pcb (KiCad board)
At the start: 2 copper layers, 100 x 50 mm, 89 parts, among them J1 Conn_01x02, J2 Conn_01x02, J3 Conn_01x03, J4 Conn_01x03, J5 Conn_01x03, J7 Conn_Coaxial, J8 Conn_Coaxial, J9 Conn_01x04, K1 HE721A0500, K2 HE721A0500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

Commit message: Update
Connections:
- net Net-(J9-Pin_2) renamed /Modules Connector/Probe_L
- net Net-(J9-Pin_3) renamed /Modules Connector/Probe_H
Routing:
- net Net-(D2-+): track 28.1 -> 42.0 mm
- net VREF2: track 108.9 -> 109.4 mm
Other:
- board text added: "0"
- board text added: "0 mm"
- board text added: "0,0000 mm / 0,0000 mm"
- board text added: "0,01 mm"
- board text added: "0,02"
- board text added: "0,035 mm"
- board text added: "0,3000 mm"
- board text added: "1"
- board text added: "1,51 mm"
- board text added: "1,6000 mm"
- board text added: "100,0000 mm x 50,0000 mm"
- board text added: "2"
- board text added: "3,3"
- board text added: "4,5"
- board text added: "B.Cu"
- board text added: "B.Mask"
- board text added: "B.Paste"
- board text added: "B.Silkscreen"
- board text added: "BOARD CHARACTERISTICS"
- board text added: "Board Thickness:"
- board text added: "Board overall dimensions:"
- board text added: "Bottom Silk Screen"
- board text added: "Bottom Solder Mask"
- board text added: "Bottom Solder Paste"
- board text added: "Castellated pads:"
- board text added: "Color"
- board text added: "Copper Finish:"
- board text added: "Copper Layer Count:"
- board text added: "Dielectric"
- board text added: "Edge card connectors:"
- board text added: "Epsilon R"
- board text added: "F.Cu"
- board text added: "F.Mask"
- board text added: "F.Paste"
- board text added: "F.Silkscreen"
- board text added: "FR4"
- board text added: "Impedance Control:"
- board text added: "Layer Name"
- board text added: "Loss Tangent"
- board text added: "Material"
- board text added: "Min hole diameter:"
- board text added: "Min track/spacing:"
- board text added: "No"
- board text added: "None"
- board text added: "Not specified"
- board text added: "Plated Board Edge:"
- board text added: "Thickness (mm)"
- board text added: "Top Silk Screen"
- board text added: "Top Solder Mask"
- board text added: "Top Solder Paste"
- board text added: "Type"
- board text added: "copper"
- board text added: "core"

Commit message: Update
Parts:
- removed H2, H3, H4: M3, MountingHole:MountingHole_3.2mm_M3_Pad
- removed R10, R24, R9: 0R, Resistor_SMD:R_0603_1608Metric
- added H5: MountingHole, MountingHole:MountingHole_3.2mm_M3, F.Cu at (105.0, 95.0)
- added H6: MountingHole, MountingHole:MountingHole_3.2mm_M3, F.Cu at (195.0, 55.0)
- added H7: MountingHole, MountingHole:MountingHole_3.2mm_M3, F.Cu at (195.0, 95.0)
Routing:
- net Net-(H4-Pad1): track 4.52 -> 0.00 mm
- net Net-(H2-Pad1): track 4.50 -> 0.00 mm
- net Net-(H3-Pad1): track 4.40 -> 0.00 mm
- net GND2: track 31.1 -> 28.6 mm, vias 221 -> 218
Other:
- outline, holes or cut-outs redrawn

Commit message: Redesign pcb
Parts:
- added C14: 1u, Capacitor_SMD:C_0603_1608Metric, F.Cu at (139.5, 59.6)
- added C16: 1u, Capacitor_SMD:C_0603_1608Metric, F.Cu at (109.5, 59.3)
- added C17: 100n, Capacitor_SMD:C_0603_1608Metric, F.Cu at (88.1, 69.2)
- added F1: 160mA, Fuse:Fuse_1206_3216Metric_Pad1.42x1.75mm_HandSolder, F.Cu at (125.5, 46.8)
- added F2: 160mA, Fuse:Fuse_1206_3216Metric_Pad1.42x1.75mm_HandSolder, F.Cu at (96.6, 46.8)
- added F3: 160mA, Fuse:Fuse_1206_3216Metric_Pad1.42x1.75mm_HandSolder, F.Cu at (105.3, 46.8)
- added J6: Conn_01x02, Connector_JST:JST_XH_B2B-XH-A_1x02_P2.50mm_Vertical, F.Cu at (104.2, 41.6)
- added RV2: MCVZ0603M180AGT, Resistor_SMD:R_0603_1608Metric_Pad0.98x0.95mm_HandSolder, F.Cu at (92.2, 51.1)
- added RV7: MCVZ0603M180AGT, Resistor_SMD:R_0603_1608Metric_Pad0.98x0.95mm_HandSolder, F.Cu at (121.4, 51.2)
- moved H6 106.8 mm to (89.1, 41.1)
- moved J1 103.4 mm to (95.6, 41.5), turned to 0 degrees
- moved C11 97.6 mm to (97.4, 60.7)
- moved D2 92.3 mm to (97.0, 50.8), turned to 0 degrees
- moved RV1 86.1 mm to (101.8, 51.1), turned to 90 degrees
- moved J9 82.4 mm to (88.8, 80.5), turned to 90 degrees
- moved C12 81.6 mm to (104.9, 59.2), turned to 90 degrees
- moved C13 79.8 mm to (107.9, 59.3), turned to 90 degrees
- moved U3 78.8 mm to (106.4, 63.9), turned to -90 degrees
- moved R25 78.4 mm to (97.1, 77.5), turned to 180 degrees
- moved R8 76.9 mm to (111.1, 59.3), turned to -90 degrees
- moved Q2 76.8 mm to (96.7, 80.1), turned to 0 degrees
- moved C15 75.7 mm to (112.7, 59.3), turned to 90 degrees
- moved H1 75.4 mm to (179.1, 41.1)
- moved R17 74.4 mm to (97.1, 82.7), turned to 180 degrees
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Connections:
- D2 pad 1: Net-(J1-Pin_2) -> Net-(J1-Pin_1)
- D2 pad 2: Net-(J1-Pin_1) -> Net-(D2-Pad2)
- D5 pad 1: Net-(J2-Pin_2) -> Net-(J2-Pin_1)
- D5 pad 2: Net-(J2-Pin_1) -> Net-(D5-Pad2)
- J9 pad 2: /Modules Connector/Probe_L -> /Modules Connector/Probe_H
- J9 pad 3: /Modules Connector/Probe_H -> /Modules Connector/Probe_L
Routing:
- net Net-(D9-A): track 16.0 -> 72.4 mm
- net VCC2: track 192.6 -> 146.3 mm, vias 3 -> 4
- net /Isolators/IN.V: track 11.0 -> 54.8 mm
- net Net-(D2-+): track 42.0 -> 1.75 mm
- net VREF2: track 109.4 -> 74.2 mm, vias 4 -> 3
- net Net-(K1-Pad7): track 37.0 -> 11.4 mm
- net Net-(K2-Pad7): track 36.4 -> 11.5 mm
- net Net-(D7-A): track 28.2 -> 49.3 mm
- net Net-(J1-Pin_1): track 5.88 -> 26.1 mm
- net Net-(D5-+): track 20.9 -> 2.07 mm
- net Net-(D2-Pad2): track 0.00 -> 17.9 mm
- net GND2: track 28.6 -> 18.1 mm, vias 218 -> 213
- net Net-(D5-Pad2): track 0.00 -> 7.99 mm
- net Net-(J2-Pin_1): track 5.16 -> 12.8 mm
- net Net-(J6-Pin_2): track 0.00 -> 5.28 mm
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- added copper zone on F.Cu, net Net-(D2-+)
- added copper zone on F.Cu, net Net-(D5-+)
Other:
- board size 100 x 50 mm -> 100 x 60.6 mm
- board text added: "S/N"

Commit message: Change R11, R13, R15 to 1u caps
Parts:
- removed R11, R13, R15: 0R, Resistor_SMD:R_0603_1608Metric
- added C24: 1u, Capacitor_SMD:C_0603_1608Metric, F.Cu at (100.8, 89.1)
- added C25: 1u, Capacitor_SMD:C_0603_1608Metric, F.Cu at (135.9, 89.1)
- added C26: 1u, Capacitor_SMD:C_0603_1608Metric, F.Cu at (170.9, 89.1)

Commit message: Bump revision to 1.1.0
Other:
- board text added: "lineScope Isolators Rev 1.1.0 03/2024"
- board text removed: "lineScope Isolators Rev 1.0.0 03/2024"
Changed lines of the file:
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@@
 	(title_block
 		(title "lineScope Isolators")
-		(date "2024-03-27")
-		(rev "1.0.0")
+		(date "2024-05-26")
+		(rev "1.1.0")
 		(company "Koszalix")
 	)
@@
 		)
 	)
-	(gr_text "lineScope Isolators\nRev 1.0.0 03/2024"
+	(gr_text "lineScope Isolators\nRev 1.1.0 03/2024"
 		(at 109.2 87.7 0)
 		(layer "F.SilkS")

Commit message: Fix C24
Parts:
- J1, J2, J6: value Conn_01x02 -> B4B-XH-A(LF)(SN)
- turned C24 to 180 degrees
