File: isolators.kicad_sch (KiCad schematic)
At the start: 16 parts, among them U1 ADuM3190, U2 ADuM3190

Commit message: Redesign pcb
Changed lines of the file:
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@@
-		)
-	)
-	(text_box "Add 2mm x 9.5mm cutout under U1,U3"
-		(exclude_from_sim no)
-		(at 142.24 73.66 0)
-		(size 22.225 5.08)
-		(stroke
-			(width 0)
-			(type default)
-		)
-		(fill
-			(type color)
-			(color 255 176 62 1)
-		)
-		(effects
-			(font
-				(size 1.27 1.27)
-			)
-			(justify left top)
 		)
 	)

Commit message: Bump revision to 1.1.0
Other:
- company: (none) -> koszalix
- title: (none) -> lineScope Isolators 
Changed lines of the file:
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@@
 	(generator_version "8.0")
 	(paper "A4")
+	(title_block
+		(title "lineScope Isolators ")
+		(date "2024-05-26")
+		(rev "Rev 1.1.0")
+		(company "koszalix")
+	)
 	(junction
 		(at 191.77 43.815)
