File: lineScope.kicad_sch (KiCad schematic)
At the start: 41 parts, among them J1 Conn_01x02, J2 Conn_Coaxial, J3 Conn_01x02, J4 Conn_Coaxial, U1 ADuM3190, U2 LM358, U3 ADuM3190

Commit message: Route pcb
Parts:
- removed C1, C7: 100n, Capacitor_SMD:C_0603_1608Metric, symbol Koszalix_Capacitors_Ceramic_Walsin_0603:CAP_100n_X7R
- removed C10, C11, C12, C2, C3, C4, C5, C6, C8, C9: 1u, Capacitor_SMD:C_0603_1608Metric, symbol Koszalix_Capacitors_Ceramic_Walsin_0603:CAP_1u_X7R
- removed D1, D2: ESD3B15WS, Diode_SMD:D_SOD-323_HandSoldering, symbol Koszalix_TVS:ESD3B15WS
- removed J1, J3: Conn_01x02, symbol Connector_Generic:Conn_01x02
- removed J2, J4: Conn_Coaxial, symbol Connector:Conn_Coaxial
- removed R1, R2, R4, R7: 10k, Resistor_SMD:R_0603_1608Metric, symbol Koszalix_Resistors_Yageo_RC0603:RES_10k_0603
- removed R10, R3, R5, R9: 1k, Resistor_SMD:R_0603_1608Metric, symbol Koszalix_Resistors_Yageo_RC0603:RES_1k_0603
- removed R6, R8: 51R, Resistor_SMD:R_0603_1608Metric, symbol Koszalix_Resistors_Yageo_RC0603:RES_51R_0603
- removed TP1, TP10, TP2, TP3, TP4, TP5, TP6, TP7, TP8, TP9: TestPoint, symbol Connector:TestPoint
- removed U1, U3: ADuM3190, symbol Koszalix_Isolators:ADuM3190
- removed U2: LM358, symbol Amplifier_Operational:LM358
Other:
- added sheet Isolators (isolators.kicad_sch)
- added sheet Modules Connector (modules_connector.kicad_sch)
- added sheet Output Drivers (drivers.kicad_sch)
- added sheet Power Supply (power_supply.kicad_sch)

Commit message: Update title frame
Other:
- company: (none) -> Koszalix
- title: (none) -> lineScope isolators
Changed lines of the file:
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@@
 	(generator_version "8.0")
 	(paper "A4")
+	(title_block
+		(title "lineScope isolators")
+		(date "2024-04-11")
+		(rev "1.0.0")
+		(company "Koszalix")
+	)
 	(wire
 		(pts

Commit message: Redesign pcb
Other:
- company: Koszalix -> (none)
- title: lineScope isolators -> (none)
Changed lines of the file:
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@@
 	(generator_version "8.0")
 	(paper "A4")
-	(title_block
-		(title "lineScope isolators")
-		(date "2024-04-11")
-		(rev "1.0.0")
-		(company "Koszalix")
-	)
 	(wire
 		(pts

Commit message: Bump revision to 1.1.0
Other:
- company: (none) -> koszalix
- title: (none) -> lineScope Isolators 
Changed lines of the file:
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@@
 	(generator_version "8.0")
 	(paper "A4")
+	(title_block
+		(title "lineScope Isolators ")
+		(date "2024-05-26")
+		(rev "Rev 1.1.0")
+		(company "koszalix")
+	)
 	(wire
 		(pts
